Commit message: ahora se puede visualizar el view.launch.py de description pero aun hay que arreglar la ubicacion del brazo

File: phantom_ws/src/phantomx_pincher/phantomx_pincher_description/urdf/phantomx_pincher.urdf.xacro (robot description, xacro)
@@ -5,6 +5,10 @@
   <!-- Imported elements -->
   <!--                   -->
+  <xacro:include filename="$(find phantomx_pincher_description)/urdf/phantomx_pincher_utils.xacro"/>
+  <xacro:include filename="$(find phantomx_pincher_description)/urdf/kit.xacro"/>
   <xacro:include filename="$(find phantomx_pincher_description)/urdf/phantomx_pincher_arm.xacro"/>
+  <!--
   <xacro:include filename="$(find phantomx_pincher_description)/urdf/phantomx_pincher_mounting.xacro"/>
+  -->
   <xacro:include filename="$(find phantomx_pincher_description)/urdf/phantomx_pincher.gazebo"/>
   <!--            -->
@@ -37,4 +41,44 @@
   <!--       -->
   <!-- Base link that can be used for fixing the robot to the world -->
+  <xacro:phantomx_pincher_dummy_link
+      link_name="$(arg prefix)${base_link}"
+      collision="$(arg collision)"
+      gazebo_preserve_fixed_joint="$(arg gazebo_preserve_fixed_joint)"/>
+  <!-- Base link -> kit "world_link" -->
+  <joint name="$(arg prefix)${base_link}_joint" type="fixed">
+    <parent link="$(arg prefix)${base_link}"/>
+    <!-- Root of the kit defined in kit.xacro -->
+    <child  link="world_link"/>
+    <origin xyz="0 0 0" rpy="0 0 0"/>
+  </joint>
+  <!-- Kit -> Arm mounting joint -->
+  <joint name="$(arg prefix)kit_to_arm_base_joint" type="fixed">
+    <!-- Parent: link from kit.xacro where the robot sits -->
+    <parent link="caseBaseRobot_link"/>
+    <!-- Child: base link of the PhantomX arm -->
+    <child  link="$(arg prefix)arm_base_link"/>
+    <!--
+      TODO: adjust xyz and rpy so that the arm base coincides
+      with the mounting holes on caseBaseRobot_link.
+      Start with zeros and tune:
+        xyz = "x y z"
+        rpy = "roll pitch yaw"
+    -->
+    <origin xyz="0 0 0" rpy="0 0 0"/>
+  </joint>
+  <!-- Arm -->
+  <xacro:phantomx_pincher
+      prefix="$(arg prefix)"
+      base_link="arm_base_link"
+      collision="$(arg collision)"
+      ros2_control="$(arg ros2_control)"
+      ros2_control_plugin="$(arg ros2_control_plugin)"
+      ros2_control_command_interface="$(arg ros2_control_command_interface)"
+      mimic_finger_joints="$(arg mimic_finger_joints)"
+      gazebo_preserve_fixed_joint="$(arg gazebo_preserve_fixed_joint)"/>
+  <!--       -->
+  <!-- Robot -->
+  <!--       -->
+  <!-- Base link that can be used for fixing the robot to the world
   <xacro:phantomx_pincher_dummy_link link_name="$(arg prefix)${base_link}" gazebo_preserve_fixed_joint="$(arg gazebo_preserve_fixed_joint)"/>
   <joint name="$(arg prefix)${base_link}_joint" type="fixed">
@@ -42,10 +86,13 @@
     <child link="$(arg prefix)task_board_link"/>
   </joint>
-  <!-- Mount -->
+   -->
+  <!-- Mount
   <xacro:task_board prefix="$(arg prefix)" child="task_board_mount_link" collision="$(arg collision)" gazebo_preserve_fixed_joint="$(arg gazebo_preserve_fixed_joint)"/>
   <xacro:task_board_mount prefix="$(arg prefix)" child="base_mount_link" collision="$(arg collision)" gazebo_preserve_fixed_joint="$(arg gazebo_preserve_fixed_joint)"/>
   <xacro:base_mount prefix="$(arg prefix)" child="arm_base_link" collision="$(arg collision)" gazebo_preserve_fixed_joint="$(arg gazebo_preserve_fixed_joint)"/>
-  <!-- Arm -->
+  -->
+  <!-- Arm
   <xacro:phantomx_pincher prefix="$(arg prefix)" base_link="arm_base_link" collision="$(arg collision)" ros2_control="$(arg ros2_control)" ros2_control_plugin="$(arg ros2_control_plugin)" ros2_control_command_interface="$(arg ros2_control_command_interface)" mimic_finger_joints="$(arg mimic_finger_joints)" gazebo_preserve_fixed_joint="$(arg gazebo_preserve_fixed_joint)"/>
+  -->
   <!-- Gazebo - ROS 2 control (Ignition) -->
   <xacro:if value="$(arg ros2_control)">

File: phantom_ws/src/phantomx_pincher/phantomx_pincher_description/urdf/phantomx_pincher_utils.xacro (robot description, xacro)
@@ -155,8 +155,7 @@
   <!-- Macro -->
   <!--       -->
-  <xacro:macro name="phantomx_pincher_dummy_link" params="
-    link_name
-    gazebo_preserve_fixed_joint:=true
-  ">
+  <xacro:macro name="phantomx_pincher_dummy_link"
+      params="link_name collision:=false gazebo_preserve_fixed_joint:=false"
+  >
     <link name="${link_name}">
       <xacro:if value="${gazebo_preserve_fixed_joint}">
